File: electronics/BackPorch/BackPorch.kicad_sch (KiCad schematic)
At the start: 15 parts, among them J1 RJ45, J2 RJ45, J3 2601-1102, J4 2601-1104, J5 2601-1104, J6 2601-1104

Commit message: Planning on ordering more back porches.
Parts:
- removed D1, D2, D3: LED, LED_SMD:LED_0603_1608Metric, symbol Device:LED
- removed H1, H2: MountingHole, MountingHole:MountingHole_3.2mm_M3, symbol Mechanical:MountingHole
- removed J1, J2: RJ45, LocalFootprints:AMPHENOL_54602-908LF, symbol Connector:RJ45
- removed J3: 2601-1102, LocalFootprints:CONN2_2601-1102_WAG, symbol LocalSyms:WAGO 2601-1102
- removed J4, J5, J6: 2601-1104, LocalFootprints:CONN4_2601-1104_WAG, symbol LocalSyms:WAGO 2601-1104
- removed R1, R2, R3: 680, Resistor_SMD:R_0603_1608Metric, symbol Device:R
- removed S1: JS202011SCQN, LocalFootprints:SW_JS202011SCQN, symbol LocalSyms:JS202011SCQN
Connections:
- no-connect marks 2 -> 0
Other:
- added sheet IO (IO.kicad_sch)
- added sheet Power (Power.kicad_sch)
- added sheet STM32 (stm32.kicad_sch)
