File: electronics/Foyers/Foyers.kicad_sch (KiCad schematic)
At the start: 11 parts, among them J1 RJ45, J2 2601-1102, J3 2601-1104

Commit message: Pulling Rev B into main (#1)
* Planning on ordering more back porches.
* Various updates to the footprints. Added datasheets.
* Added the software.
* Verified CAN, voltage input, current reading although the resistor is off, and temperature reading.
* Many updates to get things dialed in. Have the ABS signal working. But there is a small glitch to it.
* Inc encoder is now working as well.
* Added a bootloader.

* Bootloader is working to the point it can push new images into app code space.

* Refactored the CAN messages. Programming is working, at least pushing code. Build version strings are working correctly.

* Refactored the CAN messages. Programming is working, at least pushing code. Build version strings are working correctly.

* Bootblock will reboot on watchdog and stay in the bootblock.

* Forgot to add the auto increment version.

* Updated the bootblock functionality. I am able to program an app code image now.

* I can now reprogram app code from app code.

* Bootloading is working well.

* Updated the README file. It still needs some work.

* The bootblock now allows me to reprogram the bootblock.

* Many refactors to support different deviceIDs. Currently app code can't write to FLASH.

* This is mostly working.

* Things are working well. I can reprogram different units. The CAN status LED flashes as heartbeat messages come in.

* In the app added CAN bus utilization, sorted by device ID. Changed to the release build for the backporch, changed task names, moved can TX tasks into one thread and CAN Rx tasks into a second thread. Fixed a bug with the bootloader picking up the wrong device ID.

* Added the wpilib code. I have only tested the Java code and it works.
Parts:
- removed D2, D3: LED, LED_SMD:LED_0603_1608Metric_Pad1.05x0.95mm_HandSolder, symbol Device:LED
- removed R3, R4: 680, Resistor_SMD:R_0603_1608Metric_Pad0.98x0.95mm_HandSolder, symbol Device:R
